File: hardware/PCB_UNO/tirasRGB.sch (EAGLE design)
At the start: 12 parts, among them IC1 MEGA8-P, IC2 LD117AV

Commit message: Se cambia regulador del diseño PCB y se eliminan ficheros generados por la impresora de PCB
Parts:
- removed JP1, JP2: (no value), pinhead:PINHD-1X2
- removed LED1: (no value), led:LED5MM
- removed R2: (no value), rcl:R-EU_0204/5
- added +12V, +3.3V: (no value), pinhead:PINHD-1X2
- IC2: value LD117AV -> 7805T; device v-reg:LD117AV -> linear:7805T
Connections:
- removed net N$1: IC2.OUT
- removed net N$6: LED1.C, R2.2
- net 3.3V: now also +3.3V.1, IC2.VO; no longer JP1.2
- net GND: now also +12V.2, +3.3V.2, IC2.GND; no longer IC2.ADJ, JP1.1, JP2.1, R2.1
- net N$2: now also +12V.1, IC2.VI; no longer IC2.IN, JP2.2
Changed lines of the file:
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@@
 <part name="S2" library="switch-omron" deviceset="10-XX" device=""/>
 <part name="GND6" library="supply1" deviceset="GND" device=""/>
-<part name="JP1" library="pinhead" deviceset="PINHD-1X2" device=""/>
+<part name="+3.3V" library="pinhead" deviceset="PINHD-1X2" device=""/>
 <part name="GND7" library="supply1" deviceset="GND" device=""/>
-<part name="IC2" library="v-reg" deviceset="LD117A?*" device="V"/>
-<part name="LED1" library="led" deviceset="LED" device="5MM"/>
-<part name="R2" library="rcl" deviceset="R-EU_" device="0204/5"/>
-<part name="GND3" library="supply1" deviceset="GND" device=""/>
-<part name="JP2" library="pinhead" deviceset="PINHD-1X2" device=""/>
+<part name="+12V" library="pinhead" deviceset="PINHD-1X2" device=""/>
+<part name="IC2" library="linear" deviceset="78*" device="T" technology="05"/>
 </parts>
 <sheets>
@@
 <instance part="S2" gate="1" x="27.94" y="93.98"/>
 <instance part="GND6" gate="1" x="25.4" y="78.74" rot="R270"/>
-<instance part="JP1" gate="G$1" x="-10.16" y="114.3" rot="R180"/>
+<instance part="+3.3V" gate="G$1" x="-5.08" y="111.76"/>
 <instance part="GND7" gate="1" x="0" y="91.44"/>
-<instance part="IC2" gate="G$1" x="-27.94" y="114.3"/>
-<instance part="LED1" gate="G$1" x="86.36" y="43.18"/>
-<instance part="R2" gate="G$1" x="91.44" y="33.02" rot="R180"/>
-<instance part="GND3" gate="1" x="99.06" y="27.94"/>
-<instance part="JP2" gate="G$1" x="-40.64" y="91.44" rot="R270"/>
+<instance part="+12V" gate="G$1" x="-35.56" y="96.52"/>
+<instance part="IC2" gate="A1" x="-30.48" y="114.3"/>
 </instances>
 <busses>
@@
 </segment>
 <segment>
-<pinref part="JP1" gate="G$1" pin="1"/>
-<wire x1="-7.62" y1="111.76" x2="0" y2="111.76" width="0.1524" layer="91"/>
-<wire x1="0" y1="111.76" x2="0" y2="101.6" width="0.1524" layer="91"/>
-<pinref part="GND7" gate="1" pin="GND"/>
-<pinref part="IC2" gate="G$1" pin="ADJ"/>
-<wire x1="0" y1="101.6" x2="0" y2="93.98" width="0.1524" layer="91"/>
-<wire x1="-27.94" y1="93.98" x2="-27.94" y2="101.6" width="0.1524" layer="91"/>
-<wire x1="-27.94" y1="101.6" x2="-27.94" y2="106.68" width="0.1524" layer="91"/>
-<wire x1="-27.94" y1="101.6" x2="0" y2="101.6" width="0.1524" layer="91"/>
-<junction x="-27.94" y="101.6"/>
-<junction x="0" y="101.6"/>
-<pinref part="C3" gate="G$1" pin="1"/>
-<wire x1="7.62" y1="104.14" x2="7.62" y2="101.6" width="0.1524" layer="91"/>
-<wire x1="7.62" y1="101.6" x2="0" y2="101.6" width="0.1524" layer="91"/>
-<pinref part="JP2" gate="G$1" pin="1"/>
-<wire x1="-38.1" y1="93.98" x2="-27.94" y2="93.98" width="0.1524" layer="91"/>
-</segment>
-<segment>
-<pinref part="R2" gate="G$1" pin="1"/>
-<pinref part="GND3" gate="1" pin="GND"/>
-<wire x1="96.52" y1="33.02" x2="99.06" y2="33.02" width="0.1524" layer="91"/>
-<wire x1="99.06" y1="33.02" x2="99.06" y2="30.48" width="0.1524" layer="91"/>
-</segment>
-<segment>
 <pinref part="C2" gate="G$1" pin="1"/>
 <pinref part="GND2" gate="1" pin="GND"/>
@@
 <wire x1="17.78" y1="58.42" x2="12.7" y2="58.42" width="0.1524" layer="91"/>
 <junction x="12.7" y="58.42"/>
+<pinref part="GND7" gate="1" pin="GND"/>
+<wire x1="0" y1="101.6" x2="0" y2="93.98" width="0.1524" layer="91"/>
+<wire x1="-27.94" y1="101.6" x2="-5.08" y2="101.6" width="0.1524" layer="91"/>
+<junction x="0" y="101.6"/>
+<pinref part="C3" gate="G$1" pin="1"/>
+<wire x1="-5.08" y1="101.6" x2="0" y2="101.6" width="0.1524" layer="91"/>
+<wire x1="7.62" y1="104.14" x2="7.62" y2="101.6" width="0.1524" layer="91"/>
+<wire x1="7.62" y1="101.6" x2="0" y2="101.6" width="0.1524" layer="91"/>
+<pinref part="+12V" gate="G$1" pin="2"/>
+<wire x1="-38.1" y1="96.52" x2="-40.64" y2="96.52" width="0.1524" layer="91"/>
+<wire x1="-40.64" y1="96.52" x2="-40.64" y2="91.44" width="0.1524" layer="91"/>
+<wire x1="-40.64" y1="91.44" x2="-27.94" y2="91.44" width="0.1524" layer="91"/>
+<wire x1="-27.94" y1="91.44" x2="-27.94" y2="101.6" width="0.1524" layer="91"/>
+<wire x1="12.7" y1="66.04" x2="-5.08" y2="66.04" width="0.1524" layer="91"/>
+<wire x1="-5.08" y1="66.04" x2="-5.08" y2="101.6" width="0.1524" layer="91"/>
+<junction x="12.7" y="66.04"/>
+<junction x="-5.08" y="101.6"/>
+<pinref part="+3.3V" gate="G$1" pin="2"/>
+<wire x1="-7.62" y1="111.76" x2="-10.16" y2="111.76" width="0.1524" layer="91"/>
+<wire x1="-10.16" y1="111.76" x2="-10.16" y2="104.14" width="0.1524" layer="91"/>
+<wire x1="-10.16" y1="104.14" x2="0" y2="104.14" width="0.1524" layer="91"/>
+<wire x1="0" y1="104.14" x2="0" y2="101.6" width="0.1524" layer="91"/>
+<pinref part="IC2" gate="A1" pin="GND"/>
+<wire x1="-30.48" y1="106.68" x2="-30.48" y2="101.6" width="0.1524" layer="91"/>
+<wire x1="-30.48" y1="101.6" x2="-27.94" y2="101.6" width="0.1524" layer="91"/>
+<junction x="-27.94" y="101.6"/>
 </segment>
 </net>
@@
 <wire x1="12.7" y1="114.3" x2="12.7" y2="83.82" width="0.1524" layer="91"/>
 <junction x="12.7" y="83.82"/>
-<pinref part="JP1" gate="G$1" pin="2"/>
-<wire x1="-7.62" y1="114.3" x2="7.62" y2="114.3" width="0.1524" layer="91"/>
-<label x="22.86" y="114.3" size="1.778" layer="95" xref="yes"/>
 <pinref part="C3" gate="G$1" pin="2"/>
 <wire x1="7.62" y1="114.3" x2="12.7" y2="114.3" width="0.1524" layer="91"/>
-<wire x1="12.7" y1="114.3" x2="22.86" y2="114.3" width="0.1524" layer="91"/>
 <wire x1="7.62" y1="111.76" x2="7.62" y2="114.3" width="0.1524" layer="91"/>
-<junction x="7.62" y="114.3"/>
 <junction x="12.7" y="114.3"/>
-</segment>
-</net>
-<net name="N$1" class="0">
-<segment>
-<pinref part="IC2" gate="G$1" pin="OUT"/>
-<wire x1="-20.32" y1="114.3" x2="-10.16" y2="114.3" width="0.1524" layer="91"/>
+<wire x1="12.7" y1="114.3" x2="12.7" y2="121.92" width="0.1524" layer="91"/>
+<wire x1="-20.32" y1="114.3" x2="-17.78" y2="114.3" width="0.1524" layer="91"/>
+<pinref part="+3.3V" gate="G$1" pin="1"/>
+<wire x1="-17.78" y1="114.3" x2="-7.62" y2="114.3" width="0.1524" layer="91"/>
+<wire x1="12.7" y1="121.92" x2="-17.78" y2="121.92" width="0.1524" layer="91"/>
+<wire x1="-17.78" y1="121.92" x2="-17.78" y2="114.3" width="0.1524" layer="91"/>
+<junction x="-17.78" y="114.3"/>
+<pinref part="IC2" gate="A1" pin="VO"/>
 </segment>
 </net>
 <net name="N$2" class="0">
 <segment>
-<pinref part="IC2" gate="G$1" pin="IN"/>
-<wire x1="-45.72" y1="114.3" x2="-35.56" y2="114.3" width="0.1524" layer="91"/>
-<pinref part="JP2" gate="G$1" pin="2"/>
-<wire x1="-40.64" y1="93.98" x2="-45.72" y2="93.98" width="0.1524" layer="91"/>
-<wire x1="-45.72" y1="93.98" x2="-45.72" y2="114.3" width="0.1524" layer="91"/>
+<pinref part="+12V" gate="G$1" pin="1"/>
+<wire x1="-38.1" y1="99.06" x2="-45.72" y2="99.06" width="0.1524" layer="91"/>
+<wire x1="-45.72" y1="99.06" x2="-45.72" y2="114.3" width="0.1524" layer="91"/>
+<pinref part="IC2" gate="A1" pin="VI"/>
+<wire x1="-40.64" y1="114.3" x2="-45.72" y2="114.3" width="0.1524" layer="91"/>
 </segment>
 </net>
-<net name="N$6" class="0">
-<segment>
-<pinref part="LED1" gate="G$1" pin="C"/>
-<pinref part="R2" gate="G$1" pin="2"/>
-<wire x1="86.36" y1="33.02" x2="86.36" y2="38.1" width="0.1524" layer="91"/>
-</segment>
-</net>
