File: hardware/PCB_UNO/tirasRGB.sch (EAGLE design)
At the start: 17 parts, among them IC1 MEGA8-P, IC2 7805T

Commit message: Se añade sensor de sonido 3 pines
Parts:
- added SENSOR: 22-23-2031, con-molex:22-23-2031
Connections:
- new net N$12: IC1.PC5(ADC5/SCL), SENSOR-3.S
- net 3.3V: now also SENSOR-1.S
- net GND: now also SENSOR-2.S
Changed lines of the file:
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@@
 <part name="GND5" library="supply1" deviceset="GND" device=""/>
 <part name="TIRA_RGB" library="con-hirschmann" deviceset="SPB4" device=""/>
+<part name="SENSOR" library="con-molex" deviceset="22-23-2031" device=""/>
 </parts>
 <sheets>
@@
 <instance part="GND5" gate="1" x="99.06" y="45.72"/>
 <instance part="TIRA_RGB" gate="1" x="114.3" y="116.84" rot="R180"/>
+<instance part="SENSOR" gate="-1" x="58.42" y="111.76"/>
+<instance part="SENSOR" gate="-2" x="58.42" y="109.22"/>
+<instance part="SENSOR" gate="-3" x="58.42" y="106.68"/>
 </instances>
 <busses>
@@
 <wire x1="30.48" y1="99.06" x2="27.94" y2="99.06" width="0.1524" layer="91"/>
 <junction x="27.94" y="99.06"/>
+<pinref part="SENSOR" gate="-2" pin="S"/>
+<wire x1="55.88" y1="109.22" x2="38.1" y2="109.22" width="0.1524" layer="91"/>
+<wire x1="38.1" y1="109.22" x2="38.1" y2="101.6" width="0.1524" layer="91"/>
+<junction x="38.1" y="101.6"/>
 </segment>
 <segment>
@@
 <junction x="-17.78" y="114.3"/>
 <pinref part="IC2" gate="A1" pin="VO"/>
+<pinref part="SENSOR" gate="-1" pin="S"/>
+<wire x1="55.88" y1="111.76" x2="38.1" y2="111.76" width="0.1524" layer="91"/>
+<wire x1="38.1" y1="111.76" x2="38.1" y2="121.92" width="0.1524" layer="91"/>
+<wire x1="38.1" y1="121.92" x2="12.7" y2="121.92" width="0.1524" layer="91"/>
+<junction x="12.7" y="121.92"/>
 </segment>
 </net>
@@
 </segment>
 </net>
+<net name="N$12" class="0">
+<segment>
+<pinref part="SENSOR" gate="-3" pin="S"/>
+<wire x1="55.88" y1="106.68" x2="50.8" y2="106.68" width="0.1524" layer="91"/>
+<wire x1="50.8" y1="106.68" x2="50.8" y2="96.52" width="0.1524" layer="91"/>
+<wire x1="50.8" y1="96.52" x2="81.28" y2="96.52" width="0.1524" layer="91"/>
+<wire x1="81.28" y1="96.52" x2="81.28" y2="71.12" width="0.1524" layer="91"/>
+<pinref part="IC1" gate="G$1" pin="PC5(ADC5/SCL)"/>
+<wire x1="81.28" y1="71.12" x2="78.74" y2="71.12" width="0.1524" layer="91"/>
+</segment>
+</net>
