File: hardware/PCB_UNO/tirasRGB.brd (EAGLE design)
At the start: 100 x 80 mm, 17 parts, among them IC1 MEGA8-P, IC2 7805T

Commit message: Se mejora PCB de diseño
Parts:
- moved C2 1.27 mm to (24.1, 39.4)
- turned Q1 to 0 degrees
Routing:
- net N$15: track 5.08 -> 20.1 mm
- net N$14: track 8.15 -> 11.7 mm
- net GND: track 149.1 -> 147.7 mm
Changed lines of the file:
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@@
 </element>
 <element name="R1" library="rcl" package="0204/5" value="" x="16.51" y="11.43"/>
-<element name="Q1" library="crystal" package="TC26V" value="" x="22.86" y="34.29" rot="R90">
-<attribute name="OC_NEWARK" value="unknown" x="73.66" y="49.53" size="1.778" layer="27" rot="R90" display="off"/>
-<attribute name="MPN" value="" x="73.66" y="49.53" size="1.778" layer="27" rot="R90" display="off"/>
-<attribute name="MF" value="" x="73.66" y="49.53" size="1.778" layer="27" rot="R90" display="off"/>
-<attribute name="OC_FARNELL" value="unknown" x="73.66" y="49.53" size="1.778" layer="27" rot="R90" display="off"/>
+<element name="Q1" library="crystal" package="TC26V" value="" x="22.86" y="34.29">
+<attribute name="OC_NEWARK" value="unknown" x="38.1" y="-16.51" size="1.778" layer="27" display="off"/>
+<attribute name="MPN" value="" x="38.1" y="-16.51" size="1.778" layer="27" display="off"/>
+<attribute name="MF" value="" x="38.1" y="-16.51" size="1.778" layer="27" display="off"/>
+<attribute name="OC_FARNELL" value="unknown" x="38.1" y="-16.51" size="1.778" layer="27" display="off"/>
 </element>
 <element name="C1" library="capacitor-wima" package="C2.5-3" value="" x="24.13" y="27.94" rot="R180"/>
-<element name="C2" library="capacitor-wima" package="C2.5-3" value="" x="24.13" y="38.1" rot="R180"/>
+<element name="C2" library="capacitor-wima" package="C2.5-3" value="" x="24.13" y="39.37" rot="R180"/>
 <element name="C3" library="capacitor-wima" package="C2.5-3" value="" x="11.43" y="10.16" rot="R90"/>
 <element name="S2" library="switch-omron" package="B3F-10XX" value="" x="24.13" y="13.97" rot="R270">
@@
 <wire x1="26.3906" y1="17.2212" x2="26.3906" y2="24.13" width="0.8128" layer="16"/>
 <wire x1="26.3906" y1="24.13" x2="26.3906" y2="26.67" width="0.8128" layer="16"/>
-<wire x1="26.3906" y1="26.67" x2="26.3906" y2="37.1094" width="0.8128" layer="16"/>
-<wire x1="26.3906" y1="37.1094" x2="25.4" y2="38.1" width="0.8128" layer="16"/>
 <wire x1="25.4" y1="27.94" x2="25.4" y2="27.6606" width="0.8128" layer="16"/>
 <wire x1="25.4" y1="27.6606" x2="26.3906" y2="26.67" width="0.8128" layer="16"/>
@@
 <wire x1="35.56" y1="59.69" x2="34.29" y2="60.96" width="1.27" layer="16"/>
 <wire x1="34.29" y1="60.96" x2="22.86" y2="60.96" width="1.27" layer="16"/>
-<wire x1="25.4" y1="38.1" x2="25.4" y2="39.37" width="0.8128" layer="16"/>
-<wire x1="25.4" y1="39.37" x2="24.13" y2="40.64" width="0.8128" layer="16"/>
-<wire x1="24.13" y1="40.64" x2="13.97" y2="40.64" width="0.8128" layer="16"/>
-<wire x1="13.97" y1="40.64" x2="13.97" y2="55.88" width="1.27" layer="16"/>
-<wire x1="13.97" y1="55.88" x2="12.7" y2="57.15" width="1.27" layer="16"/>
+<wire x1="25.4" y1="39.37" x2="25.4" y2="27.94" width="0.8128" layer="16"/>
+<wire x1="25.4" y1="39.37" x2="22.86" y2="41.91" width="0.8128" layer="16"/>
+<wire x1="22.86" y1="41.91" x2="21.59" y2="41.91" width="0.8128" layer="16"/>
+<wire x1="21.59" y1="41.91" x2="20.32" y2="40.64" width="0.8128" layer="16"/>
+<wire x1="20.32" y1="40.64" x2="15.24" y2="40.64" width="0.8128" layer="16"/>
+<wire x1="15.24" y1="40.64" x2="12.7" y2="43.18" width="0.8128" layer="16"/>
+<wire x1="12.7" y1="43.18" x2="12.7" y2="57.15" width="0.8128" layer="16"/>
 </signal>
 <signal name="N$14">
@@
 <contactref element="C2" pad="2"/>
 <contactref element="Q1" pad="2"/>
-<wire x1="22.86" y1="38.1" x2="22.86" y2="35.56" width="0.8128" layer="16"/>
-<wire x1="22.86" y1="38.1" x2="21.59" y2="38.1" width="0.8128" layer="16"/>
-<wire x1="21.59" y1="38.1" x2="20.32" y2="36.83" width="0.8128" layer="16"/>
+<wire x1="22.86" y1="39.37" x2="20.32" y2="36.83" width="0.8128" layer="16"/>
 <wire x1="20.32" y1="36.83" x2="17.78" y2="36.83" width="0.8128" layer="16"/>
+<wire x1="24.13" y1="34.29" x2="22.86" y2="35.56" width="0.8128" layer="16"/>
+<wire x1="22.86" y1="35.56" x2="22.86" y2="39.37" width="0.8128" layer="16"/>
 </signal>
 <signal name="N$15">
@@
 <contactref element="C1" pad="2"/>
 <contactref element="Q1" pad="1"/>
+<wire x1="21.59" y1="34.29" x2="22.86" y2="33.02" width="0.8128" layer="16"/>
 <wire x1="22.86" y1="33.02" x2="22.86" y2="27.94" width="0.8128" layer="16"/>
-<wire x1="22.86" y1="33.02" x2="17.78" y2="39.37" width="0" layer="19" extent="1-1"/>
+<wire x1="21.59" y1="34.29" x2="20.32" y2="35.56" width="0.8128" layer="16"/>
+<wire x1="20.32" y1="35.56" x2="15.24" y2="35.56" width="0.8128" layer="16"/>
+<wire x1="15.24" y1="35.56" x2="15.24" y2="39.37" width="0.8128" layer="16"/>
+<wire x1="15.24" y1="39.37" x2="17.78" y2="39.37" width="0.8128" layer="16"/>
 </signal>
 <signal name="N$16">
